Commit message: tested moveit arm group

File: robotics_arm_description/urdf/robotics_arm_with_gripper.urdf (robot description, URDF)
Before this commit: robot robotics_arm, 12 links, 11 joints
Joints:
- joint gripper_base_joint: axis 0 1 0 -> 0 -1 0; origin xyz=-0.048 -0.03 0.026 rpy=3.1416 3.142 1.5708 -> xyz=-0.048 -0.03 0.026 rpy=3.142 0 1.5708
- joint joint_2: origin xyz=0 -0.019745 0.001 rpy=3.1416 3.142 -1.571 -> xyz=-0.005 -0.019745 0.001 rpy=0 3.142 -1.571
- joint joint_3: origin xyz=0.0 -0.02 -0.11 rpy=0 3.142 0 -> xyz=0.0 0.025 -0.11 rpy=0 3.142 3.142
- joint left_finger_joint: axis 0 0 1 -> 0 0 -1; limit lower=0 upper=0 effort=0 velocity=0 -> lower=0 upper=0.8 effort=0 velocity=0; mimic joint=gripper_joint multiplier=-1 offset=0 -> joint=gripper_joint multiplier=1 offset=0
- joint left_inner_joint: axis 0 0 1 -> 0 0 -1; limit lower=0 upper=0 effort=0 velocity=0 -> lower=0 upper=0.8 effort=0 velocity=0; mimic joint=gripper_joint multiplier=-1 offset=0 -> joint=gripper_joint multiplier=1 offset=0
- joint left_knuckle_joint: limit lower=0 upper=0 effort=0 velocity=0 -> lower=0 upper=0.8 effort=0 velocity=0
- joint right_inner_joint: limit lower=0 upper=0 effort=0 velocity=0 -> lower=0 upper=0.8 effort=0 velocity=0
- joint right_outer_joint: axis 0 0 1 -> 0 0 -1; limit lower=0 upper=0 effort=0 velocity=0 -> lower=0 upper=0.8 effort=0 velocity=0; mimic joint=gripper_joint multiplier=-1 offset=0 -> joint=gripper_joint multiplier=1 offset=0

File: robotics_arm_moveit/config/robotics_arm.ros2_control.xacro (robot description, xacro)
@@ -2,16 +2,16 @@
 <robot xmlns:xacro="http://www.ros.org/wiki/xacro">
     <xacro:macro name="robotics_arm_ros2_control" params="name initial_positions_file">
-        <xacro:property name="initial_positions" value="${load_yaml(initial_positions_file)['initial_positions']}"/>
+        <xacro:property name="initial_positions" value="${xacro.load_yaml(initial_positions_file)['initial_positions']}"/>
         <ros2_control name="${name}" type="system">
+          <xacro:if value="$(arg is_sim)">
+            <plugin>mock_components/GenericSystem</plugin>
+          </xacro:if>
+          <xacro:unless value="$(arg is_sim)">
             <hardware>
-                <!-- By default, set up controllers for simulation. This won't work on real hardware -->
-                <plugin>mock_components/GenericSystem</plugin>
+                <plugin>robotics_arm_control/RoboticsArm</plugin>
+                <param name="port">/dev/ttyUSB0</param>
+                <param name="baudrate">115200</param>
             </hardware>
-            <xacro:unless value="$(arg is_sim)">
-            <hardware>
-                <plugin>arduinobot_controller/ArduinobotInterface</plugin>
-                <param name="port">/dev/ttyACM0</param>
-            </hardware>
-            </xacro:unless>
+          </xacro:unless>
             <joint name="joint_1">
                 <command_interface name="position"/>
@@ -19,5 +19,4 @@
                   <param name="initial_value">${initial_positions['joint_1']}</param>
                 </state_interface>
-                <state_interface name="velocity"/>
             </joint>
             <joint name="joint_2">
@@ -26,5 +25,4 @@
                   <param name="initial_value">${initial_positions['joint_2']}</param>
                 </state_interface>
-                <state_interface name="velocity"/>
             </joint>
             <joint name="joint_3">
@@ -33,5 +31,4 @@
                   <param name="initial_value">${initial_positions['joint_3']}</param>
                 </state_interface>
-                <state_interface name="velocity"/>
             </joint>
             <joint name="joint_4">
@@ -40,5 +37,4 @@
                   <param name="initial_value">${initial_positions['joint_4']}</param>
                 </state_interface>
-                <state_interface name="velocity"/>
             </joint>
             <joint name="gripper_base_joint">
@@ -47,5 +43,4 @@
                   <param name="initial_value">${initial_positions['gripper_base_joint']}</param>
                 </state_interface>
-                <state_interface name="velocity"/>
             </joint>
             <joint name="gripper_joint">
@@ -54,5 +49,4 @@
                   <param name="initial_value">${initial_positions['gripper_joint']}</param>
                 </state_interface>
-                <state_interface name="velocity"/>
             </joint>
         </ros2_control>

File: robotics_arm_moveit/config/robotics_arm.urdf.xacro (robot description, xacro)
@@ -2,8 +2,9 @@
 <robot xmlns:xacro="http://www.ros.org/wiki/xacro" name="robotics_arm">
     <xacro:arg name="initial_positions_file" default="initial_positions.yaml" />
+    <xacro:arg name="is_sim" default="true" />
     <!-- Import robotics_arm urdf file -->
     <xacro:include filename="$(find robotics_arm_description)/urdf/robotics_arm_with_gripper.urdf" />
     <!-- Import control_xacro -->
     <xacro:include filename="robotics_arm.ros2_control.xacro" />
-    <xacro:robotics_arm_ros2_control name="FakeSystem" initial_positions_file="$(arg initial_positions_file)"/>
+    <xacro:robotics_arm_ros2_control name="ArduinoArm" initial_positions_file="$(arg initial_positions_file)"/>
 </robot>

Commit message: fixed gripper control

File: robotics_arm_description/urdf/robotics_arm_with_gripper.urdf (robot description, URDF)
Before this commit: robot robotics_arm, 12 links, 11 joints
Joints:
- joint gripper_base_joint: limit lower=0 upper=3.142 effort=0 velocity=0 -> lower=0 upper=3.142 effort=1.0 velocity=0.5
- joint gripper_joint: limit lower=0 upper=0.8 effort=0 velocity=0 -> lower=0 upper=0.8 effort=1.0 velocity=0.5
- joint joint_1: limit lower=0 upper=3.142 effort=0 velocity=0 -> lower=0 upper=3.142 effort=1.0 velocity=0.5
- joint joint_2: limit lower=0 upper=3.142 effort=0 velocity=0 -> lower=0 upper=3.142 effort=1.0 velocity=0.5
- joint joint_3: limit lower=0 upper=3.142 effort=0 velocity=0 -> lower=0 upper=3.142 effort=1.0 velocity=0.5
- joint joint_4: limit lower=0 upper=3.142 effort=0 velocity=0 -> lower=0 upper=3.142 effort=1.0 velocity=0.5
- joint left_finger_joint: limit lower=0 upper=0.8 effort=0 velocity=0 -> lower=0 upper=0.8 effort=1.0 velocity=0.5
- joint left_inner_joint: limit lower=0 upper=0.8 effort=0 velocity=0 -> lower=0 upper=0.8 effort=1.0 velocity=0.5
- joint left_knuckle_joint: limit lower=0 upper=0.8 effort=0 velocity=0 -> lower=0 upper=0.8 effort=1.0 velocity=0.5
- joint right_inner_joint: limit lower=0 upper=0.8 effort=0 velocity=0 -> lower=0 upper=0.8 effort=1.0 velocity=0.5
- joint right_outer_joint: limit lower=0 upper=0.8 effort=0 velocity=0 -> lower=0 upper=0.8 effort=1.0 velocity=0.5
